File: pcb/pcb.kicad_pcb (KiCad board)
At the start: 2 copper layers, 220.3 x 139.7 mm, 71 parts, among them J1 AudioJack3, SW1 Rotary_Encoder_Switch, SW10 Rotary_Encoder_Switch, SW2 Rotary_Encoder_Switch, SW3 Rotary_Encoder_Switch, SW4 Rotary_Encoder_Switch, SW5 Rotary_Encoder_Switch, SW6 Rotary_Encoder_Switch, SW7 Rotary_Encoder_Switch, SW8 Rotary_Encoder_Switch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

Commit message: New pcb and schematic
Parts:
- removed D44, D48: LED, LED_THT:LED_D3.0mm
- added RN1: R_Network08, Resistor_THT:R_Array_SIP9, B.Cu at (34.3, -132.7)
- added RN10: 3.3kR, Resistor_THT:R_Array_SIP9, B.Cu at (87.0, -68.6)
- added RN2: R_Network08, Resistor_THT:R_Array_SIP9, B.Cu at (72.9, -69.1)
- added RN3: R_Network08, Resistor_THT:R_Array_SIP9, B.Cu at (-46.4, -43.8)
- added RN4: R_Network08, Resistor_THT:R_Array_SIP9, B.Cu at (-36.1, -128.7)
- added RN5: R_Network08, Resistor_THT:R_Array_SIP9, B.Cu at (-90.2, -97.2)
- added RN6: 270R, Resistor_THT:R_Array_SIP9, B.Cu at (-90.2, -72.4)
- added RN7: 3.3kR, Resistor_THT:R_Array_SIP9, B.Cu at (-57.7, -88.1)
- added RN8: 3.3kR, Resistor_THT:R_Array_SIP9, B.Cu at (-70.9, -64.0)
- added RN9: 3.3kR, Resistor_THT:R_Array_SIP9, B.Cu at (69.8, -73.7)
- U7: footprint Package_DIP:DIP-8_W7.62mm_Socket -> Package_DIP:DIP-8_W7.62mm
- U8: moved to F.Cu
- moved D45 86.4 mm to (-50.8, -22.2), turned to 180 degrees
- moved U5 75.4 mm to (75.6, -73.0)
- moved U3 68.3 mm to (-28.6, -84.5), turned to 270 degrees
- moved X1 66.6 mm to (-11.4, -88.9), turned to 180 degrees
- moved U8 55.3 mm to (0.64, -118.7), turned to 0 degrees
- moved U1 41.2 mm to (-54.1, -68.8)
- moved D46 26.9 mm to (-50.8, -108.0), turned to 180 degrees
- moved U2 25.9 mm to (-2.54, -64.8), turned to 270 degrees
- moved U6 19.6 mm to (20.3, -118.7)
- moved D39 13.8 mm to (-81.8, -68.8), turned to 183.227 degrees
- moved D40 5.93 mm to (-81.3, -62.5), turned to 186.545 degrees
- moved D41 5.34 mm to (-80.4, -56.3), turned to 189.864 degrees
- moved D22 3.87 mm to (-31.9, -45.6), turned to 213.75 degrees
- moved D23 3.28 mm to (-36.8, -54.8), turned to 202.5 degrees
- moved D43 3.21 mm to (-77.5, -44.0), turned to 196.5 degrees
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Connections:
- D11 pad 2: Net-(D10-Pad2) -> Net-(D11-Pad2)
- D12 pad 2: Net-(D10-Pad2) -> Net-(D12-Pad2)
- D13 pad 2: Net-(D10-Pad2) -> Net-(D13-Pad2)
- D14 pad 2: Net-(D10-Pad2) -> Net-(D14-Pad2)
- D15 pad 2: Net-(D10-Pad2) -> Net-(D15-Pad2)
- D16 pad 2: Net-(D10-Pad2) -> Net-(D16-Pad2)
- D18 pad 2: Net-(D17-Pad2) -> Net-(D18-Pad2)
- D19 pad 2: Net-(D17-Pad2) -> Net-(D19-Pad2)
- D2 pad 2: Net-(D1-Pad2) -> Net-(D2-Pad2)
- D20 pad 2: Net-(D17-Pad2) -> Net-(D20-Pad2)
- D21 pad 2: Net-(D17-Pad2) -> Net-(D21-Pad2)
- D22 pad 2: Net-(D17-Pad2) -> Net-(D22-Pad2)
- D23 pad 2: Net-(D17-Pad2) -> Net-(D23-Pad2)
- D24 pad 2: Net-(D17-Pad2) -> Net-(D24-Pad2)
- D26 pad 2: Net-(D25-Pad2) -> Net-(D26-Pad2)
- D27 pad 2: Net-(D25-Pad2) -> Net-(D27-Pad2)
- D28 pad 2: Net-(D25-Pad2) -> Net-(D28-Pad2)
- D29 pad 2: Net-(D25-Pad2) -> Net-(D29-Pad2)
- D3 pad 2: Net-(D1-Pad2) -> Net-(D3-Pad2)
- D30 pad 2: Net-(D25-Pad2) -> Net-(D30-Pad2)
- D31 pad 2: Net-(D25-Pad2) -> Net-(D31-Pad2)
- D32 pad 2: Net-(D25-Pad2) -> Net-(D32-Pad2)
- D34 pad 2: Net-(D33-Pad2) -> Net-(D34-Pad2)
- D35 pad 2: Net-(D33-Pad2) -> Net-(D35-Pad2)
- D36 pad 2: Net-(D33-Pad2) -> Net-(D36-Pad2)
- D37 pad 2: Net-(D33-Pad2) -> Net-(D37-Pad2)
- D38 pad 2: Net-(D33-Pad2) -> Net-(D38-Pad2)
- D39 pad 1: Net-(D1-Pad1) -> Net-(D15-Pad1)
- D4 pad 2: Net-(D1-Pad2) -> Net-(D4-Pad2)
- D40 pad 1: Net-(D15-Pad1) -> Net-(D16-Pad1)
- D40 pad 2: Net-(D33-Pad2) -> Net-(D40-Pad2)
- D41 pad 1: Net-(D16-Pad1) -> Net-(D1-Pad1)
- D41 pad 2: Net-(D33-Pad2) -> Net-(D41-Pad2)
- D5 pad 2: Net-(D1-Pad2) -> Net-(D5-Pad2)
- D6 pad 2: Net-(D1-Pad2) -> Net-(D6-Pad2)
- D7 pad 2: Net-(D1-Pad2) -> Net-(D7-Pad2)
- D8 pad 2: Net-(D1-Pad2) -> Net-(D8-Pad2)
- D9 pad 2: Net-(D10-Pad2) -> Net-(D9-Pad2)
- SW1 pad S1: Net-(SW1-PadS1) -> Net-(RN8-Pad7)
- SW2 pad A: Net-(SW2-PadA) -> Net-(RN9-Pad4)
- SW2 pad B: Net-(SW2-PadB) -> Net-(RN10-Pad7)
- SW3 pad S1: Net-(SW3-PadS1) -> Net-(RN8-Pad8)
- SW4 pad A: Net-(SW4-PadA) -> Net-(RN9-Pad5)
- SW4 pad B: Net-(SW4-PadB) -> Net-(RN10-Pad6)
- SW6 pad A: Net-(SW6-PadA) -> Net-(RN9-Pad6)
- SW6 pad B: Net-(SW6-PadB) -> Net-(RN10-Pad5)
- SW9 pad S1: Net-(SW9-PadS1) -> Net-(RN8-Pad9)
- U1 pad 26: Net-(SW2-PadB) -> Net-(RN7-Pad7)
- U1 pad 27: Net-(SW4-PadB) -> Net-(RN7-Pad8)
- U1 pad 28: Net-(SW6-PadB) -> Net-(RN7-Pad9)
- U1 pad 6: Net-(SW2-PadA) -> Net-(RN8-Pad7)
- U1 pad 7: Net-(SW4-PadA) -> Net-(RN8-Pad8)
- U1 pad 8: Net-(SW6-PadA) -> Net-(RN8-Pad9)
- U5 pad 20: Net-(U5-Pad20) -> Net-(A1-Pad5)
- U5 pad 23: Net-(U5-Pad23) -> Net-(RN10-Pad7)
- U5 pad 24: Net-(U5-Pad24) -> Net-(RN10-Pad6)
- U5 pad 25: Net-(U5-Pad25) -> Net-(RN10-Pad5)
- U5 pad 3: Net-(SW1-PadS1) -> Net-(RN9-Pad4)
- U5 pad 4: Net-(SW3-PadS1) -> Net-(RN9-Pad5)
- U5 pad 5: Net-(U5-Pad5) -> Net-(RN9-Pad6)
- U6 pad 11: Net-(A1-Pad16) -> Net-(U6-Pad11)
- U6 pad 12: Net-(A1-Pad9) -> Net-(U6-Pad12)
- U6 pad 14: Net-(A1-Pad14) -> Net-(U6-Pad14)
- U8 pad 1: Net-(D10-Pad2) -> Net-(RN2-Pad1)
- U8 pad 11: Net-(A1-Pad16) -> Net-(U6-Pad11)
- U8 pad 12: Net-(A1-Pad9) -> Net-(U6-Pad12)
- U8 pad 15: Net-(D1-Pad2) -> Net-(RN1-Pad1)
- U8 pad 2: Net-(D17-Pad2) -> Net-(RN3-Pad1)
- U8 pad 3: Net-(D25-Pad2) -> Net-(RN4-Pad1)
- U8 pad 4: Net-(D33-Pad2) -> Net-(RN5-Pad1)
Routing:
- net +5V: track 1.77 -> 236.6 mm, vias 0 -> 5
- net Net-(A1-Pad23): track 0.00 -> 218.5 mm, vias 0 -> 5
- net Net-(A1-Pad24): track 0.00 -> 211.1 mm, vias 0 -> 5
- net GND: track 0.00 -> 188.7 mm, vias 0 -> 5
- net Net-(RN3-Pad1): track 0.00 -> 165.5 mm, vias 0 -> 2
- net Net-(RN6-Pad1): track 0.00 -> 163.8 mm
- net Net-(RN2-Pad1): track 0.00 -> 139.7 mm
- net Net-(RN5-Pad1): track 0.00 -> 139.1 mm
- net Net-(D1-Pad2): track 161.7 -> 26.5 mm
- net Net-(D10-Pad2): track 139.0 -> 6.67 mm
- net Net-(D12-Pad1): track 245.8 -> 376.6 mm, vias 0 -> 4
- net Net-(A1-Pad5): track 0.00 -> 123.5 mm, vias 0 -> 1
- net Net-(D14-Pad1): track 316.8 -> 418.5 mm, vias 0 -> 4
- net Net-(D15-Pad1): track 315.1 -> 410.9 mm, vias 0 -> 4
- net Net-(D33-Pad2): track 110.6 -> 18.0 mm
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Other:
- board size 220.3 x 139.7 mm -> 204.1 x 125 mm
- rule via_min_size: 0.4 -> 0.6
