File: pcb/pcb.sch (KiCad schematic (older format))
At the start: 71 parts, among them J1 AudioJack3, SW1 Rotary_Encoder_Switch, SW10 Rotary_Encoder_Switch, SW2 Rotary_Encoder_Switch, SW3 Rotary_Encoder_Switch, SW4 Rotary_Encoder_Switch, SW5 Rotary_Encoder_Switch, SW6 Rotary_Encoder_Switch, SW7 Rotary_Encoder_Switch, SW8 Rotary_Encoder_Switch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

Commit message: New pcb and schematic
Parts:
- added RN1, RN2, RN3, RN4, RN5: R_Network08, Resistor_THT:R_Array_SIP9, symbol Device:R_Network08
- added RN10, RN7, RN8, RN9: 3.3kR, Resistor_THT:R_Array_SIP9, symbol Device:R_Network08
- added RN6: 270R, Resistor_THT:R_Array_SIP9, symbol Device:R_Network08
Connections:
- net +5V: now also RN7.1 (common), RN8.1 (common), RN9.1 (common)
- net at A1.14 (D11), U2.14 (SER): no longer U6.14 (SER)
- net at A1.16 (D13), U2.11 (SRCLK): no longer U6.11 (SRCLK), U8.11 (SRCLK)
- net at A1.5 (D2): now also U5.20 (INTA)
- net at A1.9 (D6), U2.12 (RCLK): no longer U6.12 (RCLK), U8.12 (RCLK)
- net at SW1.A, U1.1 (GPB0): now also RN8.2 (R1)
- net at SW3.A, U1.2 (GPB1): now also RN8.3 (R2)
- net at SW1.B, U1.21 (GPA0): now also RN7.2 (R1)
- net at SW3.B, U1.22 (GPA1): now also RN7.3 (R2)
- net at SW5.B, U1.23 (GPA2): now also RN7.4 (R3)
- net at SW7.B, U1.24 (GPA3): now also RN7.5 (R4)
- net at SW9.B, U1.25 (GPA4): now also RN7.6 (R5)
- net at U1.26 (GPA5): now also RN7.7 (R6); no longer SW2.B
- net at U1.27 (GPA6): now also RN7.8 (R7); no longer SW4.B
- net at U1.28 (GPA7): now also RN7.9 (R8); no longer SW6.B
- net at SW5.A, U1.3 (GPB2): now also RN8.4 (R3)
- net at SW7.A, U1.4 (GPB3): now also RN8.5 (R4)
- net at SW9.A, U1.5 (GPB4): now also RN8.6 (R5)
- net at U1.6 (GPB5): now also SW1.S1, RN8.7 (R6); no longer SW2.A
- net at U1.7 (GPB6): now also SW3.S1, RN8.8 (R7); no longer SW4.A
- net at U1.8 (GPB7): now also SW9.S1, RN8.9 (R8); no longer SW6.A
- net at SW8.A, U5.1 (GPB0): now also RN9.2 (R1)
- net at SW10.A, U5.2 (GPB1): now also RN9.3 (R2)
- net at SW8.B, U5.21 (GPA0): now also RN10.9 (R8)
- net at SW10.B, U5.22 (GPA1): now also RN10.8 (R7)
- net at U5.23 (GPA2): now also SW2.B, RN10.7 (R6)
- net at U5.24 (GPA3): now also SW4.B, RN10.6 (R5)
- net at U5.25 (GPA4): now also SW6.B, RN10.5 (R4)
- net at U5.26 (GPA5): now also RN10.4 (R3)
- net at U5.27 (GPA6): now also RN10.3 (R2)
- net at U5.28 (GPA7): now also RN10.2 (R1)
- net at U5.3 (GPB2): now also SW2.A, RN9.4 (R3); no longer SW1.S1
- net at U5.4 (GPB3): now also SW4.A, RN9.5 (R4); no longer SW3.S1
- net at U5.5 (GPB4): now also SW6.A, RN9.6 (R5)
- net at U5.6 (GPB5): now also RN9.7 (R6)
- net at U5.7 (GPB6): now also RN9.8 (R7)
- net at U5.8 (GPB7): now also RN9.9 (R8)
- net at D1.1 (K), D17.1 (K), D25.1 (K)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: now also D41.1 (K); no longer D39.1 (K)
- net at D39.2 (A): now also RN5.8 (R7)
- net at D15.1 (K), D23.1 (K), D31.1 (K)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: now also D39.1 (K); no longer D40.1 (K)
- net at D16.1 (K), D24.1 (K), D32.1 (K)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: now also D40.1 (K); no longer D41.1 (K)
- net at U8.5 (QF): now also RN6.1 (common)
- net at D42.2 (A): now also RN6.3 (R2)
- net at D43.2 (A): now also RN6.4 (R3)
- net at D44.2 (A): now also RN6.5 (R4)
- net at D45.2 (A): now also RN6.6 (R5)
- net at D46.2 (A): now also RN6.7 (R6)
- net at D47.2 (A): now also RN6.8 (R7)
- net at D48.2 (A): now also RN6.9 (R8)
- new net: D1.2 (A), RN1.2 (R1)
- new net: U6.11 (SRCLK), U8.11 (SRCLK)
- new net: U6.12 (RCLK), U8.12 (RCLK)
- new net: RN2.1 (common), U8.1 (QB)
- new net: RN1.1 (common), U8.15 (QA)
- new net: RN3.1 (common), U8.2 (QC)
- new net: RN4.1 (common), U8.3 (QD)
- new net: RN5.1 (common), U8.4 (QE)
- new net: D2.2 (A), RN1.3 (R2)
- new net: D3.2 (A), RN1.4 (R3)
- new net: D4.2 (A), RN1.5 (R4)
- new net: D5.2 (A), RN1.6 (R5)
- new net: D6.2 (A), RN1.7 (R6)
- new net: D7.2 (A), RN1.8 (R7)
- new net: D8.2 (A), RN1.9 (R8)
- new net: D9.2 (A), RN2.2 (R1)
- new net: D10.2 (A), RN2.3 (R2)
- new net: D11.2 (A), RN2.4 (R3)
- new net: D16.2 (A), RN2.9 (R8)
- new net: D15.2 (A), RN2.8 (R7)
- new net: D14.2 (A), RN2.7 (R6)
- new net: D13.2 (A), RN2.6 (R5)
- new net: D12.2 (A), RN2.5 (R4)
- new net: D17.2 (A), RN3.2 (R1)
- new net: D18.2 (A), RN3.3 (R2)
- new net: D19.2 (A), RN3.4 (R3)
- new net: D24.2 (A), RN3.9 (R8)
- new net: D23.2 (A), RN3.8 (R7)
- new net: D22.2 (A), RN3.7 (R6)
- new net: D21.2 (A), RN3.6 (R5)
- new net: D20.2 (A), RN3.5 (R4)
- new net: D25.2 (A), RN4.2 (R1)
- new net: D26.2 (A), RN4.3 (R2)
- new net: D27.2 (A), RN4.4 (R3)
- new net: D32.2 (A), RN4.9 (R8)
- new net: D31.2 (A), RN4.8 (R7)
- new net: D30.2 (A), RN4.7 (R6)
- new net: D29.2 (A), RN4.6 (R5)
- new net: D28.2 (A), RN4.5 (R4)
- new net: D33.2 (A), RN5.2 (R1)
- new net: D34.2 (A), RN5.3 (R2)
- new net: D35.2 (A), RN5.4 (R3)
- new net: D40.2 (A), RN5.9 (R8)
- new net: D38.2 (A), RN5.7 (R6)
- new net: D37.2 (A), RN5.6 (R5)
- new net: D36.2 (A), RN5.5 (R4)
- new net: D41.2 (A), RN6.2 (R1)
Other:
- moved on the sheet: A1, C1, C2, D1, D2, D3, D4, D5, D6, D7, D8, J1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
